File: layout/st_ekg_v1/st_ekg_v1.brd (EAGLE design)
At the start: 59.4 x 56.8 mm, 31 parts, among them J1 SJ1-3523N

Commit message: Add photos of layout and schematics
Parts:
- added R15: 1Meg, rcl:M0805
Connections:
- net GND: now also R15.1
- net N$22: now also R15.2
Routing:
- net N$22: track 3.94 -> 7.44 mm
Changed lines of the file:
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@@
 <attribute name="VALUE" x="6.35" y="57.15" size="1.27" layer="27" rot="R180"/>
+</element>
+<element name="R15" library="rcl" library_urn="urn:adsk.eagle:library:334" package="M0805" package3d_urn="urn:adsk.eagle:package:23556/2" value="1Meg" x="33.3375" y="8.255" smashed="yes" rot="MR180">
+<attribute name="NAME" x="32.0675" y="6.985" size="1.27" layer="26" rot="MR180"/>
+<attribute name="POPULARITY" value="45" x="33.3375" y="8.255" size="1.778" layer="28" rot="MR180" display="off"/>
+<attribute name="SPICEPREFIX" value="R" x="33.3375" y="8.255" size="1.778" layer="28" rot="MR180" display="off"/>
+<attribute name="VALUE" x="32.0675" y="10.795" size="1.27" layer="28" rot="MR180"/>
 </element>
 </elements>
@@
 <vertex x="0" y="0"/>
 </polygon>
+<contactref element="R15" pad="1"/>
 </signal>
 <signal name="N$4">
@@
 <signal name="N$7">
 <contactref element="IC1" pad="12"/>
-<contactref element="R5" pad="2"/>
 <contactref element="R11" pad="1"/>
 <wire x1="45.4025" y1="41.275" x2="51.755" y2="41.275" width="0.8128" layer="16"/>
-<wire x1="42.5425" y1="27.305" x2="46.355" y2="27.305" width="0.8128" layer="1"/>
-<wire x1="46.355" y1="27.305" x2="51.7525" y2="32.7025" width="0.8128" layer="1"/>
+<wire x1="51.7525" y1="32.7025" x2="46.355" y2="27.305" width="0.8128" layer="1"/>
 <via x="51.7525" y="32.7025" extent="1-16" drill="0.9"/>
 <wire x1="51.7525" y1="32.7025" x2="51.7525" y2="41.2725" width="0.8128" layer="16"/>
 <wire x1="51.7525" y1="41.2725" x2="51.755" y2="41.275" width="0.8128" layer="16"/>
+<contactref element="R5" pad="2"/>
+<wire x1="46.355" y1="27.305" x2="42.5425" y2="27.305" width="0.8128" layer="1"/>
 </signal>
 <signal name="N$8">
@@
 <wire x1="40.0075" y1="7.935" x2="41.5925" y2="7.935" width="0.8128" layer="16"/>
 <wire x1="39.6875" y1="8.255" x2="40.0075" y2="7.935" width="0.8128" layer="16"/>
+<contactref element="R15" pad="2"/>
+<wire x1="37.7825" y1="8.255" x2="34.2875" y2="8.255" width="0.8128" layer="16"/>
 </signal>
 <signal name="N$23">
